Commit message: Fixed URDF base_link

File: models/basic_rmp.urdf (robot description, URDF)
Before this commit: robot rmp_401, 2 links, 1 joints
Links:
- link base_link: geometry collision box size=${base_length} ${base_width} ${base_height}; visual mesh filename=package://mcity_proxy/meshes/chassis.stl scale=0.001 0.001 0.001

Commit message: Working version of URDF complete

File: models/basic_rmp.urdf (robot description, URDF)
Before this commit: robot rmp_401, 2 links, 1 joints
Links:
- added link base_footprint
- added link front_steer_link; visual mesh filename=package://mcity_proxy/meshes/steering_arm.stl scale=0.001 0.001 0.001
- link gps_link: geometry visual box size=.042 .05 .001
Joints:
- added joint base_joint: type fixed, parent base_footprint, child base_link, origin xyz=0.0 0.0 ${(wheel_radius+wheel_zoff)} rpy=0 0 0
- added joint steer_joint: type revolute, parent base_link, child front_steer_link, origin xyz=0 0.22 0 rpy=0 0 0, axis 0 0 1, limit lower=-0.36 upper=0.36 effort=30 velocity=5.0
- joint gps_joint: origin xyz=0.10 0 0.05 rpy=0 0 0 -> xyz=-0.01 -.117 0.08 rpy=0 0 0

Commit message: Gazebo working

File: models/basic_rmp.urdf (robot description, URDF)
Before this commit: robot rmp_401, 4 links, 3 joints
Links:
- added link backwhl_l_link, mass 1; collision cylinder length=0.085 radius=0.1075; visual mesh filename=/home/luckierdodge/dev_ws/install/mcity_proxy/share/mcity_p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 scale=0.001 0.001 0.001
- added link backwhl_r_link, mass 1; collision cylinder length=0.085 radius=0.1075; visual mesh filename=/home/luckierdodge/dev_ws/install/mcity_proxy/share/mcity_p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 scale=0.001 0.001 0.001
- added link frontwhl_l_link, mass 1; collision cylinder length=0.085 radius=0.1075; visual mesh filename=/home/luckierdodge/dev_ws/install/mcity_proxy/share/mcity_p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 scale=0.001 0.001 0.001
- added link frontwhl_r_link, mass 1; collision cylinder length=0.085 radius=0.1075; visual mesh filename=/home/luckierdodge/dev_ws/install/mcity_proxy/share/mcity_p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 scale=0.001 0.001 0.001
- link base_link: mass None -> 20.0; geometry collision box size=0.432 0.635 0.204; visual mesh filename=/home/luckierdodge/dev_ws/install/mcity_proxy/share/mcity_p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 scale=0.001 0.001 0.001
- link front_steer_link: mass None -> 5.0; geometry visual mesh filename=/home/luckierdodge/dev_ws/install/mcity_proxy/share/mcity_p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 scale=0.001 0.001 0.001
Joints:
- added joint backwhl_l_joint: type continuous, parent base_link, child backwhl_l_link, origin xyz=-0.24 -.235 -.09 rpy=0 0 3.14159265359, axis 1 0 0
- added joint backwhl_r_joint: type continuous, parent base_link, child backwhl_r_link, origin xyz=0.24 -.235 -.09 rpy=0 0 0, axis 1 0 0
- added joint frontwhl_l_joint: type continuous, parent front_steer_link, child frontwhl_l_link, origin xyz=-0.22 0 -.09 rpy=0 0 3.14159265359, axis 1 0 0
- added joint frontwhl_r_joint: type continuous, parent front_steer_link, child frontwhl_r_link, origin xyz=0.22 0 -.09 rpy=0 0 0, axis 1 0 0
- joint base_joint: origin xyz=0.0 0.0 ${(wheel_radius+wheel_zoff)} rpy=0 0 0 -> xyz=0.0 0.0 0.1575 rpy=0 0 0
