Commit message: Add zed camera; fix x-axis forward issue

File: models/basic_rmp.urdf.xacro (robot description, xacro)
@@ -54,5 +54,5 @@
   <link name="base_link">
     <visual>
-      <origin xyz="-.355 -.3450 -.200" rpy="1.5707963267949 0 0"/>
+      <origin xyz="-.3450 .355 -.200" rpy="${pi/2} 0 -${pi/2}"/>
       <geometry>
         <mesh filename="file://$(find mcity_proxy)/meshes/chassis.stl" scale="0.001 0.001 0.001"/>
@@ -64,8 +64,8 @@
     <collision>
       <geometry>
-        <box size="${base_width} ${base_length} ${base_height}"/>
+        <box size="${base_length} ${base_width} ${base_height}"/>
       </geometry>
     </collision>
-    <xacro:box_inertia m="20.0" w="${base_width}" d="${base_length}" h="${base_height}" xyz="0 0 0" rpy="${pi/2} 0 0"/>
+    <xacro:box_inertia m="20.0" w="${base_length}" d="${base_width}" h="${base_height}" xyz="0 0 0" rpy="${pi/2} 0 -${pi/2}"/>
   </link>
   <gazebo reference="base_link">
@@ -75,5 +75,5 @@
   <link name="front_steer_link">
     <visual>
-      <origin xyz="-.355 -.5650 -.200" rpy="1.5707963267949 0 0"/>
+      <origin xyz="-.5650 .355 -.200" rpy="1.5707963267949 0 -${pi/2}"/>
       <geometry>
         <mesh filename="file://$(find mcity_proxy)/meshes/steering_arm.stl" scale="0.001 0.001 0.001"/>
@@ -88,5 +88,5 @@
     <parent link="base_link"/>
     <child link="front_steer_link"/>
-    <origin xyz="0 0.22 0" rpy="0 0 0"/>
+    <origin xyz="0.22 0 0" rpy="0 0 0"/>
     <limit upper="0.36" lower="-0.36" effort="30" velocity="5.0"/>
     <axis xyz="0 0 1"/>
@@ -99,5 +99,5 @@
     <link name="${prefix}_link">
       <visual>
-        <origin xyz="${-.355 - offset_multiplier * x_offset} -.5650 -.110" rpy="1.5707963267949 0 0"/>
+        <origin xyz="-.5650 ${.355 + offset_multiplier * x_offset} -.110" rpy="1.5707963267949 0 -${pi/2}"/>
         <geometry>
           <mesh filename="file://$(find mcity_proxy)/meshes/front_wheel.stl" scale="0.001 0.001 0.001"/>
@@ -108,19 +108,16 @@
       </visual>
       <collision>
-        <origin xyz=".048 0 0" rpy="0 ${pi/2} 0"/>
-        <!-- <origin xyz="${-.355 - offset_multiplier * x_offset} -.5650 -.110" rpy="1.5707963267949 0 0"/> -->
+        <origin xyz="0 .048 0" rpy="0 ${pi/2} ${-pi/2}"/>
         <geometry>
           <cylinder radius="${wheel_radius}" length="${wheel_width}"/>
         </geometry>
       </collision>
-      <xacro:cylinder_inertia m="1" r="${wheel_radius}" h="${wheel_width}" xyz=".048 0 0" rpy="0 ${pi/2} 0"/>
+      <xacro:cylinder_inertia m="1" r="${wheel_radius}" h="${wheel_width}" xyz=".048 0 0" rpy="0 ${pi/2} ${-pi/2}"/>
     </link>
     <joint name="${prefix}_joint" type="continuous">
       <parent link="front_steer_link"/>
       <child link="${prefix}_link"/>
-      <!-- <origin xyz="${x_reflect*wheel_xoff} ${y_reflect*(base_width/2+wheel_ygap)} ${-wheel_zoff}" rpy="0 0 0"/> -->
-      <origin xyz="${x_offset} 0 -.09" rpy="0 0 ${z_rotate}"/>
-      <!-- <limit upper="3.1415" lower="-3.1415" effort="30" velocity="5.0"/> -->
-      <axis xyz="${offset_multiplier * -1} 0 0"/>
+      <origin xyz="0 ${x_offset} -.09" rpy="0 0 ${z_rotate}"/>
+      <axis xyz="0 ${offset_multiplier} 0"/>
     </joint>
     <gazebo reference="${prefix}_link">
@@ -128,11 +125,11 @@
     </gazebo>
   </xacro:macro>
-  <xacro:front_wheel prefix="frontwhl_r" x_offset=".22" offset_multiplier="1" z_rotate="0"/>
-  <xacro:front_wheel prefix="frontwhl_l" x_offset="-.22" offset_multiplier="-1" z_rotate="3.14159265359"/>
+  <xacro:front_wheel prefix="frontwhl_r" x_offset=".22" offset_multiplier="-1" z_rotate="0"/>
+  <xacro:front_wheel prefix="frontwhl_l" x_offset="-.22" offset_multiplier="1" z_rotate="${pi}"/>
   <!-- ***********************  BACK WHEELS ******************************  -->
   <xacro:macro name="back_wheel" params="prefix x_offset offset_multiplier z_rotate">
     <link name="${prefix}_link">
       <visual>
-        <origin xyz="${-.355 - offset_multiplier * x_offset} -.1100 -.110" rpy="1.5707963267949 0 0"/>
+        <origin xyz="-.1100 ${.355 + offset_multiplier * x_offset} -.110" rpy="1.5707963267949 0 -${pi/2}"/>
         <geometry>
           <mesh filename="file://$(find mcity_proxy)/meshes/back_wheel.stl" scale="0.001 0.001 0.001"/>
@@ -143,18 +140,16 @@
       </visual>
       <collision>
-        <origin xyz=".029 0 0" rpy="0 ${pi/2} 0"/>
+        <origin xyz="0 .029 0" rpy="0 ${pi/2} -${pi/2}"/>
         <geometry>
           <cylinder radius="${wheel_radius}" length="${wheel_width}"/>
         </geometry>
       </collision>
-      <xacro:cylinder_inertia m="1" r="${wheel_radius}" h="${wheel_width}" xyz=".029 0 0" rpy="0 ${pi/2} 0"/>
+      <xacro:cylinder_inertia m="1" r="${wheel_radius}" h="${wheel_width}" xyz=".029 0 0" rpy="0 ${pi/2} ${-pi/2}"/>
     </link>
     <joint name="${prefix}_joint" type="continuous">
       <parent link="base_link"/>
       <child link="${prefix}_link"/>
-      <!-- <origin xyz="${x_reflect*wheel_xoff} ${y_reflect*(base_width/2+wheel_ygap)} ${-wheel_zoff}" rpy="0 0 0"/> -->
-      <origin xyz="${x_offset} -.235 -.09" rpy="0 0 ${z_rotate}"/>
-      <!-- <limit upper="3.1415" lower="-3.1415" effort="30" velocity="5.0"/> -->
-      <axis xyz="1 0 0"/>
+      <origin xyz="-.235 ${x_offset} -.09" rpy="0 0 ${z_rotate}"/>
+      <axis xyz="0 ${offset_multiplier} 0"/>
     </joint>
     <gazebo reference="${prefix}_link">
@@ -162,11 +157,11 @@
     </gazebo>
   </xacro:macro>
-  <xacro:back_wheel prefix="backwhl_r" x_offset=".24" offset_multiplier="1" z_rotate="0"/>
-  <xacro:back_wheel prefix="backwhl_l" x_offset="-.24" offset_multiplier="-1" z_rotate="3.14159265359"/>
+  <xacro:back_wheel prefix="backwhl_r" x_offset=".24" offset_multiplier="-1" z_rotate="0"/>
+  <xacro:back_wheel prefix="backwhl_l" x_offset="-.24" offset_multiplier="1" z_rotate="3.14159265359"/>
   <!-- *********************** GPS SETUP **********************************  -->
   <link name="gps_link">
     <visual>
       <geometry>
-        <box size=".042 .05 .001"/>
+        <box size=".05 .042 .001"/>
       </geometry>
       <material name="Blue">
@@ -174,10 +169,10 @@
       </material>
     </visual>
-    <xacro:box_inertia m="0.1" w=".042" d=".05" h=".001" xyz="0 0 0" rpy="0 0 0"/>
+    <xacro:box_inertia m="0.1" w=".05" d=".042" h=".001" xyz="0 0 0" rpy="0 0 0"/>
   </link>
   <joint name="gps_joint" type="fixed">
     <parent link="base_link"/>
     <child link="gps_link"/>
-    <origin xyz="-0.01 -.117 0.08" rpy="0 0 0"/>
+    <origin xyz="-.117 0.01 0.08" rpy="0 0 0"/>
   </joint>
   <gazebo reference="gps_link">
@@ -209,7 +204,4 @@
     </sensor>
   </gazebo>
-  <!-- <gazebo reference="base_joint">
-    <preserveFixedJoint>true</preserveFixedJoint>
-  </gazebo> -->
   <!-- *********************** IMU SETUP *********************************  -->
   <!-- Each sensor must be attached to a link.                              -->
@@ -217,5 +209,5 @@
     <visual>
       <geometry>
-        <box size=".042 .05 .001"/>
+        <box size=".05 .042 .001"/>
       </geometry>
       <material name="Blue">
@@ -223,5 +215,5 @@
       </material>
     </visual>
-    <xacro:box_inertia m="0.1" w=".042" d=".05" h=".001" xyz="0 0 0" rpy="0 0 0"/>
+    <xacro:box_inertia m="0.1" w=".05" d=".042" h=".001" xyz="0 0 0" rpy="0 0 0"/>
   </link>
   <joint name="imu_joint" type="fixed">
@@ -308,41 +300,133 @@
     </sensor>
   </gazebo>
-<!-- *********************** WHEEL ODOMETRY ***************************    -->
-<gazebo>
-  <plugin name="rmp_drive_controller" filename="libgazebo_ros_diff_drive.so">
-    <ros>
-      <!-- Set namespace -->
-      <namespace>/</namespace>
-      <!-- Remap default topics -->
-      <!-- <remapping>cmd_vel:=cmd_demo</remapping> -->
-      <remapping>odom:=odometry/wheel</remapping>
-    </ros>
-    <!-- Update rate -->
-    <update_rate>500</update_rate>
-    <!-- Number of wheel pairs -->
-    <num_wheel_pairs>2</num_wheel_pairs>
-    <!-- wheels0 -->
-    <left_joint>frontwhl_l_joint</left_joint>
-    <right_joint>frontwhl_r_joint</right_joint>
-    <!-- wheels1-->
-    <left_joint>backwhl_r_joint</left_joint>
-    <right_joint>backwhl_r_joint</right_joint>
-    <!-- kinematics -->
-    <wheel_separation>0.55</wheel_separation>
-    <wheel_separation>0.55</wheel_separation>
-    <wheel_diameter>0.215</wheel_diameter>
-    <wheel_diameter>0.215</wheel_diameter>
-    <!-- limits -->
-    <max_wheel_torque>20</max_wheel_torque>
-    <max_wheel_acceleration>1.0</max_wheel_acceleration>
-    <!-- output -->
-    <publish_odom>true</publish_odom>
-    <publish_odom_tf>true</publish_odom_tf>
-    <!-- <publish_wheel_tf>true</publish_wheel_tf> -->
-    <!-- <odometry_frame>odom_demo</odometry_frame> -->
-    <robot_base_frame>base_footprint</robot_base_frame>
-  </plugin>
-</gazebo>
- <!-- *********************** JOINT STATE PUBLISHER *********************   -->
+  <!-- *********************** ZED 2i SENSOR  ***************************    -->
+  <link name="camera_link">
+    <visual>
+      <geometry>
+        <mesh filename="file://$(find mcity_proxy)/meshes/zed_2i.stl" scale="0.001 0.001 0.001"/>
+      </geometry>
+      <material name="Blue">
+        <color rgba="${0/255} ${0/255} ${255/255} 1.0"/>
+      </material>
+      <origin xyz="-0.05 .01 0" rpy="0 0 ${pi/2}"/>
+    </visual>
+    <xacro:box_inertia m="0.224" w=".175" d=".3" h=".43" xyz="0 0 0" rpy="0 0 0"/>
+  </link>
+  <joint name="camera_joint" type="fixed">
+    <parent link="base_link"/>
+    <child link="camera_link"/>
+    <origin xyz="0.3 0 0.095" rpy="0 0 0"/>
+  </joint>
+  <joint name="camera_optical_joint" type="fixed">
+    <!-- these values have to be these values otherwise the gazebo camera
+        image won't be aligned properly with the frame it is supposedly
+        originating from -->
+    <origin xyz="0 0 0" rpy="${-pi/2} 0 ${-pi/2}"/>
+    <parent link="camera_link"/>
+    <child link="camera_link_optical"/>
+  </joint>
+  <link name="camera_link_optical">
+    <xacro:box_inertia m="0.01" w=".01" d=".01" h=".01" xyz="0 0 0" rpy="0 0 0"/>
+  </link>
+  <gazebo reference="camera_link">
+    <sensor type="depth" name="zed_2i">
+        <!-- Set always_on only sensor, not on plugin -->
+        <always_on>1</always_on>
+        <!-- Set update_rate only sensor, not on plugin -->
+        <update_rate>1</update_rate>
+        <camera name="zed_2i">
+          <distortion>
+            <!-- TODO Fix distortion params -->
+            <k1>0.1</k1>
+            <k2>0.2</k2>
+            <k3>0.3</k3>
+            <p1>0.4</p1>
+            <p2>0.5</p2>
+            <center>0.5 0.5</center>
+          </distortion>
+          <horizontal_fov>1.26</horizontal_fov>
+            <image>
+              <width>1920</width>
+              <height>1080</height>
+              <format>B8G8R8</format>
+            </image>
+            <depth_camera>
+            </depth_camera>
+            <clip>
+              <near>0.02</near>
+              <far>300</far>
+            </clip>
+            <noise>
+              <type>gaussian</type>
+              <!-- Noise is sampled independently per pixel on each frame.
+                   That pixel's noise value is added to each of its color
+                   channels, which at that point lie in the range [0,1]. -->
+              <mean>0.0</mean>
+              <stddev>0.007</stddev>
+            </noise>
+        </camera>
+        <plugin name="zed_2i_depth_camera" filename="libgazebo_ros_camera.so">
+          <!-- Change namespace, camera name and topics so -
+                * Raw images are published to /custom_ns/custom_camera/custom_image
+                * Depth images are published to /custom_ns/custom_camera/custom_image_depth
+                * Raw image camera info is published to /custom_ns/custom_camera/custom_info_raw
+                * Depth image camera info is published to /custom_ns/custom_camera/custom_info_depth
+                * Point cloud is published to /custom_ns/custom_camera/custom_points
+          -->
+          <ros>
+            <namespace>/</namespace>
+            <remapping>depth_cam/image_raw:=custom_camera/custom_image</remapping>
+            <remapping>depth_cam/image_depth:=custom_camera/custom_image_depth</remapping>
+            <remapping>depth_cam/camera_info:=custom_camera/custom_info_raw</remapping>
+            <remapping>depth_cam/camera_info_depth:=custom_camera/custom_info_depth</remapping>
+            <remapping>depth_cam/points:=custom_camera/custom_points</remapping>
+          </ros>
+          <!-- Set camera name. If empty, defaults to sensor name (i.e. "sensor_name") -->
+          <camera_name>zed_2i</camera_name>
+          <!-- Set TF frame name. If empty, defaults to link name (i.e. "link_name") -->
+          <frame_name>camera_link_optical</frame_name>
+          <hack_baseline>0.12</hack_baseline>
+          <!-- No need to repeat distortion parameters or to set autoDistortion -->
+          <min_depth>1.5</min_depth>
+          <max_depth>35</max_depth>
+      </plugin>
+    </sensor>
+  </gazebo>
+  <!-- *********************** WHEEL ODOMETRY ***************************    -->
+  <gazebo>
+    <plugin name="rmp_drive_controller" filename="libgazebo_ros_diff_drive.so">
+      <ros>
+        <!-- Set namespace -->
+        <namespace>/</namespace>
+        <!-- Remap default topics -->
+        <remapping>odom:=odometry/wheel</remapping>
+      </ros>
+      <!-- Update rate -->
+      <update_rate>500</update_rate>
+      <!-- Number of wheel pairs -->
+      <num_wheel_pairs>2</num_wheel_pairs>
+      <!-- wheels0 -->
+      <left_joint>frontwhl_l_joint</left_joint>
+      <right_joint>frontwhl_r_joint</right_joint>
+      <!-- wheels1-->
+      <left_joint>backwhl_r_joint</left_joint>
+      <right_joint>backwhl_r_joint</right_joint>
+      <!-- kinematics -->
+      <wheel_separation>0.55</wheel_separation>
+      <wheel_separation>0.55</wheel_separation>
+      <wheel_diameter>0.215</wheel_diameter>
+      <wheel_diameter>0.215</wheel_diameter>
+      <!-- limits -->
+      <max_wheel_torque>20</max_wheel_torque>
+      <max_wheel_acceleration>1.0</max_wheel_acceleration>
+      <!-- output -->
+      <publish_odom>true</publish_odom>
+      <publish_odom_tf>true</publish_odom_tf>
+      <!-- <publish_wheel_tf>true</publish_wheel_tf> -->
+      <!-- <odometry_frame>odom_demo</odometry_frame> -->
+      <robot_base_frame>base_footprint</robot_base_frame>
+    </plugin>
+  </gazebo>
+  <!-- *********************** JOINT STATE PUBLISHER *********************   -->
   <gazebo>
     <plugin name="rmp_joint_state" filename="libgazebo_ros_joint_state_publisher.so">

Commit message: Babysteps towards navstack working

File: models/basic_rmp.urdf.xacro (robot description, xacro)
@@ -48,7 +48,4 @@
     <origin xyz="0.0 0.0 ${(wheel_radius+wheel_zoff)}" rpy="0 0 0"/>
   </joint>
-  <!-- <gazebo reference="base_joint">
-    <preserveFixedJoint>true</preserveFixedJoint>
-  </gazebo> -->
   <!-- ********************** ROBOT BASE *********************************  -->
   <link name="base_link">
@@ -119,5 +116,5 @@
       <child link="${prefix}_link"/>
       <origin xyz="0 ${x_offset} -.09" rpy="0 0 ${z_rotate}"/>
-      <axis xyz="0 ${offset_multiplier} 0"/>
+      <axis xyz="0 ${-1 * offset_multiplier} 0"/>
     </joint>
     <gazebo reference="${prefix}_link">
@@ -151,5 +148,5 @@
       <child link="${prefix}_link"/>
       <origin xyz="-.235 ${x_offset} -.09" rpy="0 0 ${z_rotate}"/>
-      <axis xyz="0 ${offset_multiplier} 0"/>
+      <axis xyz="0 ${-1 * offset_multiplier} 0"/>
     </joint>
     <gazebo reference="${prefix}_link">
@@ -335,4 +332,5 @@
         <!-- Set update_rate only sensor, not on plugin -->
         <update_rate>1</update_rate>
+        <visualize>true</visualize>
         <camera name="zed_2i">
           <distortion>
@@ -376,9 +374,9 @@
           <ros>
             <namespace>/</namespace>
-            <remapping>depth_cam/image_raw:=custom_camera/custom_image</remapping>
+            <!-- <remapping>depth_cam/image_raw:=custom_camera/custom_image</remapping>
             <remapping>depth_cam/image_depth:=custom_camera/custom_image_depth</remapping>
             <remapping>depth_cam/camera_info:=custom_camera/custom_info_raw</remapping>
             <remapping>depth_cam/camera_info_depth:=custom_camera/custom_info_depth</remapping>
-            <remapping>depth_cam/points:=custom_camera/custom_points</remapping>
+            <remapping>depth_cam/points:=custom_camera/custom_points</remapping> -->
           </ros>
           <!-- Set camera name. If empty, defaults to sensor name (i.e. "sensor_name") -->
@@ -426,4 +424,8 @@
       <!-- <odometry_frame>odom_demo</odometry_frame> -->
       <robot_base_frame>base_footprint</robot_base_frame>
+      <!-- Odometry source, 0 for ENCODER, 1 for WORLD, defaults to WORLD -->
+      <odometry_source>1</odometry_source>
+      <odometry_topic>odom</odometry_topic>
+      <odometry_frame>odom</odometry_frame>
     </plugin>
   </gazebo>

Commit message: Fixes for turning; parameter tuning

File: models/basic_rmp.urdf.xacro (robot description, xacro)
@@ -82,9 +82,9 @@
     <xacro:box_inertia m="5.0" w=".46" d=".09" h=".20" xyz="0 0 0" rpy="0 0 0"/>
   </link>
-  <joint name="steer_joint" type="revolute">
+  <joint name="steer_joint" type="fixed">
     <parent link="base_link"/>
     <child link="front_steer_link"/>
     <origin xyz="0.22 0 0" rpy="0 0 0"/>
-    <limit upper="0.36" lower="-0.36" effort="30" velocity="5.0"/>
+    <!-- <limit upper="0.36" lower="-0.36" effort="30" velocity="5.0"/> -->
     <axis xyz="0 0 1"/>
   </joint>
@@ -96,5 +96,5 @@
     <link name="${prefix}_link">
       <visual>
-        <origin xyz="-.5650 ${.355 + offset_multiplier * x_offset} -.110" rpy="1.5707963267949 0 -${pi/2}"/>
+        <origin xyz="-.5650 ${.355 - offset_multiplier * x_offset} -.110" rpy="1.5707963267949 0 -${pi/2}"/>
         <geometry>
           <mesh filename="file://$(find mcity_proxy)/meshes/front_wheel.stl" scale="0.001 0.001 0.001"/>
@@ -115,6 +115,6 @@
       <parent link="front_steer_link"/>
       <child link="${prefix}_link"/>
-      <origin xyz="0 ${x_offset} -.09" rpy="0 0 ${z_rotate}"/>
-      <axis xyz="0 ${-1 * offset_multiplier} 0"/>
+      <origin xyz="0 ${-x_offset} -.09" rpy="0 0 ${z_rotate}"/>
+      <axis xyz="0 ${-offset_multiplier} 0"/>
     </joint>
     <gazebo reference="${prefix}_link">
@@ -128,5 +128,5 @@
     <link name="${prefix}_link">
       <visual>
-        <origin xyz="-.1100 ${.355 + offset_multiplier * x_offset} -.110" rpy="1.5707963267949 0 -${pi/2}"/>
+        <origin xyz="-.1100 ${.355 - offset_multiplier * x_offset} -.110" rpy="1.5707963267949 0 -${pi/2}"/>
         <geometry>
           <mesh filename="file://$(find mcity_proxy)/meshes/back_wheel.stl" scale="0.001 0.001 0.001"/>
@@ -147,6 +147,6 @@
       <parent link="base_link"/>
       <child link="${prefix}_link"/>
-      <origin xyz="-.235 ${x_offset} -.09" rpy="0 0 ${z_rotate}"/>
-      <axis xyz="0 ${-1 * offset_multiplier} 0"/>
+      <origin xyz="-.235 ${-x_offset} -.09" rpy="0 0 ${z_rotate}"/>
+      <axis xyz="0 ${-offset_multiplier} 0"/>
     </joint>
     <gazebo reference="${prefix}_link">
@@ -416,6 +416,6 @@
       <wheel_diameter>0.215</wheel_diameter>
       <!-- limits -->
-      <max_wheel_torque>20</max_wheel_torque>
-      <max_wheel_acceleration>1.0</max_wheel_acceleration>
+      <max_wheel_torque>50</max_wheel_torque>
+      <max_wheel_acceleration>2.0</max_wheel_acceleration>
       <!-- output -->
       <publish_odom>true</publish_odom>

Commit message: Latest nav2 work

File: models/basic_rmp.urdf.xacro (robot description, xacro)
@@ -82,9 +82,10 @@
     <xacro:box_inertia m="5.0" w=".46" d=".09" h=".20" xyz="0 0 0" rpy="0 0 0"/>
   </link>
-  <joint name="steer_joint" type="fixed">
+  <joint name="steer_joint" type="revolute">
     <parent link="base_link"/>
     <child link="front_steer_link"/>
     <origin xyz="0.22 0 0" rpy="0 0 0"/>
-    <!-- <limit upper="0.36" lower="-0.36" effort="30" velocity="5.0"/> -->
+    <limit upper="0.36" lower="-0.36" effort="1" velocity="5.0"/>
+    <joint_properties damping="1.0" friction="1.0"/>
     <axis xyz="0 0 1"/>
   </joint>
@@ -117,7 +118,21 @@
       <origin xyz="0 ${-x_offset} -.09" rpy="0 0 ${z_rotate}"/>
       <axis xyz="0 ${-offset_multiplier} 0"/>
+      <joint_properties damping="1.0" friction="1.0"/>
     </joint>
     <gazebo reference="${prefix}_link">
       <material>Gazebo/White</material>
+      <collision>
+        <friction>
+          <mu1>1.4</mu1>
+          <mu2>1.4</mu2>
+          <fdir1>1 0 0</fdir1>
+          <kp>1000000.0</kp>
+          <kd>100.0</kd>
+          <minDepth>0.01</minDepth>
+          <maxContacts>1</maxContacts>
+          <slip1>1.0</slip1>
+          <slip2>0.0</slip2>
+        </friction>
+      </collision>
     </gazebo>
   </xacro:macro>
@@ -149,7 +164,21 @@
       <origin xyz="-.235 ${-x_offset} -.09" rpy="0 0 ${z_rotate}"/>
       <axis xyz="0 ${-offset_multiplier} 0"/>
+      <joint_properties damping="1.0" friction="1.0"/>
     </joint>
     <gazebo reference="${prefix}_link">
       <material>Gazebo/White</material>
+      <collision>
+        <friction>
+          <mu1>1.4</mu1>
+          <mu2>1.4</mu2>
+          <fdir1>1 0 0</fdir1>
+          <kp>1000000.0</kp>
+          <kd>100.0</kd>
+          <minDepth>0.01</minDepth>
+          <maxContacts>1</maxContacts>
+          <slip1>1.0</slip1>
+          <slip2>0.0</slip2>
+        </friction>
+      </collision>
     </gazebo>
   </xacro:macro>
@@ -416,6 +445,6 @@
       <wheel_diameter>0.215</wheel_diameter>
       <!-- limits -->
-      <max_wheel_torque>50</max_wheel_torque>
-      <max_wheel_acceleration>2.0</max_wheel_acceleration>
+      <max_wheel_torque>1000</max_wheel_torque>
+      <max_wheel_acceleration>10.0</max_wheel_acceleration>
       <!-- output -->
       <publish_odom>true</publish_odom>
@@ -428,4 +457,7 @@
       <odometry_topic>odom</odometry_topic>
       <odometry_frame>odom</odometry_frame>
+      <covariance_x>0.001</covariance_x> <!-- 0.0001 -->
+      <covariance_y>0.001</covariance_y> <!-- 0.0001 -->
+      <covariance_yaw>0.01</covariance_yaw> <!-- 0.01 -->
     </plugin>
   </gazebo>

Commit message: Fixing GPS/Odom bugs, implemented status msgs

File: models/basic_rmp.urdf.xacro (robot description, xacro)
@@ -186,5 +186,5 @@
   <xacro:back_wheel prefix="backwhl_l" x_offset="-.24" offset_multiplier="1" z_rotate="3.14159265359"/>
   <!-- *********************** GPS SETUP **********************************  -->
-  <link name="gps_link">
+  <link name="gps">
     <visual>
       <geometry>
@@ -199,8 +199,8 @@
   <joint name="gps_joint" type="fixed">
     <parent link="base_link"/>
-    <child link="gps_link"/>
+    <child link="gps"/>
     <origin xyz="-.117 0.01 0.08" rpy="0 0 0"/>
   </joint>
-  <gazebo reference="gps_link">
+  <gazebo reference="gps">
     <material>Gazebo/Blue</material>
     <sensor name="rmp_gps" type="gps">
